Commit message: feat(urdf): add pillow joint

File: src/basic_robot_pkg/urdf/robot_simplified.urdf.xacro (robot description, xacro)
@@ -262,8 +262,10 @@
     <material>Gazebo/Green</material>
 </gazebo>
-<joint name="base_link_to_mobile_frame" type="fixed">
+<joint name="base_link_to_mobile_frame" type="prismatic">
     <parent link="base_link"/>
     <child link="mobile_frame"/>
     <origin xyz="${baseDepth/2.0 + mobileFrameDepth/2.0} 0.0 ${-baseHeight/2.0 + mobileFrameHeight/2.0}"/>
+    <axis xyz="0 0 1"/>
+    <limit lower="0" upper="0.10" effort="${ELEVATION_MAX_EFFORT}" velocity="${ELEVATION_MAX_VELOCITY}"/>
 </joint>
 <gazebo reference="base_link_to_mobile_frame">
@@ -326,8 +328,10 @@
     <material>Gazebo/Black</material>
 </gazebo>
-<joint name="trolley_top_to_trolley_bottom" type="fixed">
+<joint name="trolley_top_to_trolley_bottom" type="prismatic">
     <parent link="trolley_top"/>
     <child link="trolley_bottom"/>
     <origin xyz="${-distanceFromTrolleyTopToTrolleyBottom} 0.0 0.0"/>
+    <axis xyz="0 0 -1" />
+    <limit lower="0" upper="0.1" effort="${ELEVATION_MAX_EFFORT}" velocity="${ELEVATION_MAX_VELOCITY}" />
 </joint>
 <gazebo reference="trolley_top_to_trolley_bottom">
@@ -582,4 +586,24 @@
   </actuator>
 </transmission>
+<transmission name="pillow_front">
+  <type>transmission_interface/SimpleTransmission</type>
+  <joint name="base_link_to_mobile_frame">
+    <hardwareInterface>PositionJointInterface</hardwareInterface>
+  </joint>
+  <actuator name="motor7">
+    <hardwareInterface>PositionJointInterface</hardwareInterface>
+    <mechanicalReduction>1</mechanicalReduction>
+  </actuator>
+</transmission>
+<transmission name="pillow_back">
+  <type>transmission_interface/SimpleTransmission</type>
+  <joint name="trolley_top_to_trolley_bottom">
+    <hardwareInterface>PositionJointInterface</hardwareInterface>
+  </joint>
+  <actuator name="motor8">
+    <hardwareInterface>PositionJointInterface</hardwareInterface>
+    <mechanicalReduction>1</mechanicalReduction>
+  </actuator>
+</transmission>
 <transmission name="central_cylinder">
   <type>transmission_interface/SimpleTransmission</type>

Commit message: fix(urdf): oriantation of the virtual wheel was wrong

File: src/basic_robot_pkg/urdf/robot_simplified.urdf.xacro (robot description, xacro)
@@ -511,5 +511,5 @@
   <parent link="base_link" />
   <child link="virtual_middle_engine" />
-  <axis xyz="0 0 1" />
+  <axis xyz="0 1 0" />
   <limit lower="${-maxInt}" upper="${maxInt}" effort="${DIRECTION_MAX_EFFORT}" velocity="${DIRECTION_MAX_VELOCITY}" />
 </joint>
@@ -517,5 +517,5 @@
     <origin xyz="0 0 0" rpy="0 0 0" />
     <visual>
-        <origin xyz="0 0 0" rpy="0 0 0" />
+        <origin xyz="0 0 0" rpy="${PI/2} 0 0" />
         <geometry>
             <cylinder radius="${wheelRadius}" length="${wheelWidth}"/>
@@ -524,5 +524,5 @@
     </visual>
     <inertial>
-        <origin xyz="0 0.0 0" rpy="0 0 0" />
+        <origin xyz="0 0.0 0" rpy="${PI/2} 0 0" />
         <mass value="0.01" />
         <inertia ixx="0" ixy="0" ixz="0" iyy="0" iyz="0" izz="0"/>

Commit message: fix(extend): The extend no longer disturb the power wheel control

File: src/basic_robot_pkg/urdf/robot_simplified.urdf.xacro (robot description, xacro)
@@ -56,5 +56,5 @@
     <xacro:property name="DIRECTION_MAX_EFFORT" value="10000000000"/>
     <xacro:property name="ELEVATION_MAX_EFFORT" value="40000"/>
-    <xacro:property name="ELEVATION_MAX_VELOCITY" value="1"/>
+    <xacro:property name="ELEVATION_MAX_VELOCITY" value="0.1"/>
     <xacro:property name="EXTEND_MAX_EFFORT" value="1000000"/>
     <xacro:property name="EXTEND_MAX_VELOCITY" value="0.06"/>
@@ -589,8 +589,8 @@
   <type>transmission_interface/SimpleTransmission</type>
   <joint name="base_link_to_mobile_frame">
-    <hardwareInterface>PositionJointInterface</hardwareInterface>
+    <hardwareInterface>VelocityJointInterface</hardwareInterface>
   </joint>
   <actuator name="motor7">
-    <hardwareInterface>PositionJointInterface</hardwareInterface>
+    <hardwareInterface>VelocityJointInterface</hardwareInterface>
     <mechanicalReduction>1</mechanicalReduction>
   </actuator>
@@ -599,8 +599,8 @@
   <type>transmission_interface/SimpleTransmission</type>
   <joint name="trolley_top_to_trolley_bottom">
-    <hardwareInterface>PositionJointInterface</hardwareInterface>
+    <hardwareInterface>VelocityJointInterface</hardwareInterface>
   </joint>
   <actuator name="motor8">
-    <hardwareInterface>PositionJointInterface</hardwareInterface>
+    <hardwareInterface>VelocityJointInterface</hardwareInterface>
     <mechanicalReduction>1</mechanicalReduction>
   </actuator>

Commit message: fix(urdf): sens of rotation was wrong for steer and power

File: src/basic_robot_pkg/urdf/robot_simplified.urdf.xacro (robot description, xacro)
@@ -134,5 +134,5 @@
     <child link="bottom_motor_left"/>
     <origin xyz="0.0 ${-baseWidth/2.0 - wheelRadius} ${-baseHeight/2.0 - distanceToTheGround + wheelRadius + bottomMotorHeight/2.0}"/>
-    <axis xyz="0 0 1"/>
+    <axis xyz="0 0 -1"/>
     <limit lower="${-maxInt}" upper="${maxInt}" effort="${DIRECTION_MAX_EFFORT}" velocity="${DIRECTION_MAX_VELOCITY}" />
 </joint>
@@ -167,5 +167,5 @@
     <child link="left_wheel"/>
     <origin xyz="0.0 0.0 ${-bottomMotorHeight/2.0}"/>
-    <axis xyz="0 1 0"/>
+    <axis xyz="0 -1 0"/>
     <limit lower="0" upper="0" effort="${PROPULSION_MAX_EFFORT}" velocity="${PROPULSION_MAX_VELOCITY}" />
 </joint>
@@ -200,5 +200,5 @@
     <child link="bottom_motor_right"/>
     <origin xyz="0.0 ${baseWidth/2.0 + wheelRadius} ${-baseHeight/2.0 - distanceToTheGround + wheelRadius + bottomMotorHeight/2.0}"/>
-    <axis xyz="0 0 1"/>
+    <axis xyz="0 0 -1"/>
     <limit lower="${-maxInt}" upper="${maxInt}" effort="${DIRECTION_MAX_EFFORT}" velocity="${DIRECTION_MAX_VELOCITY}" />
 </joint>
@@ -233,5 +233,5 @@
     <child link="right_wheel"/>
     <origin xyz="0.0 0.0 ${-bottomMotorHeight/2.0}"/>
-    <axis xyz="0 1 0"/>
+    <axis xyz="0 -1 0"/>
     <limit lower="0" upper="0" effort="${PROPULSION_MAX_EFFORT}" velocity="${PROPULSION_MAX_VELOCITY}" />
 </joint>
@@ -511,5 +511,5 @@
   <parent link="base_link" />
   <child link="virtual_middle_engine" />
-  <axis xyz="0 1 0" />
+  <axis xyz="0 -1 0" />
   <limit lower="${-maxInt}" upper="${maxInt}" effort="${DIRECTION_MAX_EFFORT}" velocity="${DIRECTION_MAX_VELOCITY}" />
 </joint>

Commit message: fix(urdf): virtual middle wheel and virtual wheel axes

File: src/basic_robot_pkg/urdf/robot_simplified.urdf.xacro (robot description, xacro)
@@ -511,5 +511,5 @@
   <parent link="base_link" />
   <child link="virtual_middle_engine" />
-  <axis xyz="0 -1 0" />
+  <axis xyz="0 0 -1" />
   <limit lower="${-maxInt}" upper="${maxInt}" effort="${DIRECTION_MAX_EFFORT}" velocity="${DIRECTION_MAX_VELOCITY}" />
 </joint>
@@ -533,5 +533,5 @@
   <parent link="virtual_middle_engine" />
   <child link="virtual_middle_wheel" />
-  <axis xyz="0 1 0" />
+  <axis xyz="0 -1 0" />
   <limit lower="0" upper="0" effort="${PROPULSION_MAX_EFFORT}" velocity="${PROPULSION_MAX_VELOCITY}" />
 </joint>
